Commit message: Update mobile_robot.urdf.xacro

File: urdf/mobile_robot.urdf.xacro (robot description, xacro)
@@ -1,3 +1,12 @@
 <?xml version="1.0"?>
+<robot name="mobile_robot" xmlns:xacro="http://www.ros.org/wiki/xacro">
+	<material name="blue"> <color rgba="0.0 0.0 1.0 1"/></material>
+	<material name="red"> <color rgba="1.0 0.0 0.0 1"/></material>
+	<material name="black"> <color rgba="0.1 0.1 0.1 1"/></material>
+	<link name="base_footprint"/>
+	<joint name="base_footprint_joint" type="fixed">
+		<parent link = "base_footprint"/>
+		<child link = "chassis"/>
+		<origin xyz="0 0 0.06" rpy="0 0 0"/><?xml version="1.0"?>
 <robot name="mobile_robot" xmlns:xacro="http://www.ros.org/wiki/xacro">
 	<material name="blue"> <color rgba="0.0 0.0 1.0 1"/></material>
@@ -75,4 +84,47 @@
 		<origin xyz="0 0 0.075" rpy="0 0 0"/>
 	</joint>
+	<link name ="imu_link">
+		<inertial>
+			<mass value="0.01"/>
+				<inertia ixx="0.00001" ixy="0" ixz="0"
+					 iyy="0.00001" iyz="0"
+					 izz="0.00001"/>
+		</inertial>
+		<visual>
+			<geometry><box size="0.03 0.03 0.01"/></geometry>
+			<material name="black"/>
+		</visual>
+	</link>
+	<joint name="imu_joint" type="fixed">
+		<parent link="chassis"/>
+		<child link="imu_link"/>
+		<origin xyz="0 0 0.06" rpy="0 0 0"/>
+	</joint>
+	<link name="camera_link">
+		<inertial>
+			<mass value="0.05"/>
+			<inertia ixx="0.00001" ixy="0" ixz="0"
+				 iyy="0.00001" iyz="0"
+				 izz="0.00001"/>
+		</inertial>
+		<visual>
+			<geometry><box size="0.04 0.06 0.04"/></geometry>
+			<material name="black"/>
+		</visual>
+		<collision>
+			<geometry><box size="0.04 0.06 0.04"/></geometry>
+		</collision>
+	</link>
+	<joint name="camera_joint" type="fixed">
+		<parent link="chassis"/>
+		<child link="camera_link"/>
+		<origin xyz="0.225 0 0.02" rpy="0 0 0"/>
+	</joint>
+	<link name="camera_optical_link"/>
+	<joint name="camera_optical_joint" type="fixed">
+		<parent link="camera_link"/>
+		<child link="camera_optical_link"/>
+		<origin xyz="0 0 0" rpy="${-pi/2} 0 ${-pi/2}"/>
+	</joint>
 	<gazebo reference="lidar_frame">
 		<sensor name="lidar" type="gpu_lidar">
@@ -104,4 +156,51 @@
 		</sensor>
 	</gazebo>
+	<gazebo reference="imu_link">
+		<sensor name="imu_sensor" type="imu">
+			<always_on>true</always_on>
+			<update_rate>100</update_rate>
+			<visualize>true</visualize>
+			<topic>imu</topic>
+			<gz_frame_id>imu_link</gz_frame_id>
+			<imu>
+				<angular_velocity>
+					<x><noise type="gaussian"><mean>0</mean><stddev>0.009</stddev></noise></x>
+					<y><noise type="gaussian"><mean>0</mean><stddev>0.009</stddev></noise></y>
+					<z><noise type="gaussian"><mean>0</mean><stddev>0.009</stddev></noise></z>
+				</angular_velocity>
+				<linear_acceleration>
+					<x><noise type="gaussian"><mean>0</mean><stddev>0.1</stddev></noise></x>
+					<y><noise type="gaussian"><mean>0</mean><stddev>0.1</stddev></noise></y>
+					<z><noise type="gaussian"><mean>0</mean><stddev>0.1</stddev></noise></z>
+				</linear_acceleration>
+			</imu>
+		</sensor>
+	</gazebo>
+	<gazebo reference="camera_link">
+		<sensor name="camera_link" type="camera">
+			<always_on>true</always_on>
+			<update_rate>30</update_rate>
+			<visualize>true</visualize>
+			<topic>camera/image_raw</topic>
+			<gz_frame_id>camera_optical_link</gz_frame_id>
+			<camera>
+				<horizontal_fov>1.047</horizontal_fov>
+				<image>
+					<width>640</width>
+					<height>480</height>
+					<format>R8G8B8</format>
+				</image>
+				<clip>
+					<near>0.1</near>
+					<far>100</far>
+				</clip>
+				<noise>
+					<type>gaussian</type>
+					<mean>0.0</mean>
+					<stddev>0.007</stddev>
+				</noise>
+			</camera>
+		</sensor>
+	</gazebo>
 	<gazebo>
 		<plugin filename="gz-sim-diff-drive-system" name="gz::sim::systems::DiffDrive">
@@ -141,2 +240,134 @@
 	<xacro:wheel_gazebo name="rear_right_wheel"/>
 </robot>
+	</joint>
+	<link name="chassis">
+		<inertial>
+			<mass value="2"/>
+			<inertia ixx="0.03375" ixy="0" ixz="0"
+				 iyy="0.015"   iyz="0"
+				 izz="0.04875"/>
+		</inertial>
+		<visual>
+			<geometry><box size="0.45 0.3 0.12"/></geometry>
+			<material name="blue"/>
+		</visual>
+		<collision>
+			<geometry><box size="0.45 0.3 0.12"/></geometry>
+		</collision>
+	</link>
+	<xacro:macro name="wheel" params="name x y">
+		<link name = "${name}">
+			<inertial>
+				<mass value="1"/>
+				<inertia ixx="0.000975" ixy="0" ixz="0"
+					 iyy="0.000975" iyz="0"
+					 izz="0.0018"/>
+			</inertial>
+			<visual>
+				<origin xyz="0 0 0" rpy="1.5707963 0 0"/>
+				<geometry><cylinder radius="0.06" length="0.03"/></geometry>
+				<material name="red"/>
+			</visual>
+			<collision>
+				<origin xyz="0 0 0" rpy="1.5707963 0 0"/>
+				<geometry><cylinder radius="0.06" length="0.03"/></geometry>
+			</collision>
+		</link>
+		<joint name="${name}_joint" type="continuous">
+			<parent link="chassis"/>
+			<child link="${name}"/>
+			<origin xyz="${x} ${y} -0.06" rpy="0 0 0"/>
+			<axis xyz="0 1 0"/>
+			<dynamics damping="0.05" friction="0.05"/>
+		</joint>
+	</xacro:macro>
+	<xacro:wheel name="front_left_wheel" x=" 0.12" y=" 0.165"/>
+	<xacro:wheel name="rear_left_wheel" x="-0.12" y=" 0.165"/>
+	<xacro:wheel name="front_right_wheel" x=" 0.12" y="-0.165"/>
+	<xacro:wheel name="rear_right_wheel" x="-0.12" y="-0.165"/>
+	<link name="lidar_frame">
+		<inertial>
+			<mass value="0.1"/>
+			<inertia ixx="0.000975" ixy="0" ixz="0"
+				 iyy="0.000975" iyz="0"
+				 izz="0.0018"/>
+		</inertial>
+		<visual>
+			<geometry><cylinder radius="0.04" length="0.03"/></geometry>
+			<material name="black"/>
+		</visual>
+		<collision>
+			<geometry><cylinder radius="0.04" length="0.03"/></geometry>
+		</collision>
+	</link>
+	<joint name="lidar_frame_joint" type="fixed">
+		<parent link="chassis"/>
+		<child link="lidar_frame"/>
+		<origin xyz="0 0 0.075" rpy="0 0 0"/>
+	</joint>
+	<gazebo reference="lidar_frame">
+		<sensor name="lidar" type="gpu_lidar">
+			<pose>0 0 0 0 0 0</pose>
+			<visualize>true</visualize>
+			<update_rate>10</update_rate>
+			<lidar>
+				<scan>
+					<horizontal>
+						<samples>360</samples>
+						<resolution>1</resolution>
+						<min_angle>-3.14159</min_angle>
+						<max_angle>3.14159</max_angle>
+					</horizontal>
+				</scan>
+				<range>
+					<min>0.3</min>
+					<max>12.0</max>
+					<resolution>0.01</resolution>
+				</range>
+				<noise>
+					<type>gaussian</type>
+					<mean>0.0</mean>
+					<stddev>0.01</stddev>
+				</noise>
+			</lidar>
+			<topic>scan</topic>
+			<gz_frame_id>lidar_frame</gz_frame_id>
+		</sensor>
+	</gazebo>
+	<gazebo>
+		<plugin filename="gz-sim-diff-drive-system" name="gz::sim::systems::DiffDrive">
+			<left_joint>front_left_wheel_joint</left_joint>
+			<left_joint>rear_left_wheel_joint</left_joint>
+			<right_joint>front_right_wheel_joint</right_joint>
+			<right_joint>rear_right_wheel_joint</right_joint>
+			<wheel_separation>0.48</wheel_separation>
+			<wheel_radius>0.06</wheel_radius>
+			<topic>/cmd_vel</topic>
+			<odom_topic>/odom</odom_topic>
+			<frame_id>odom</frame_id>
+			<child_frame_id>base_footprint</child_frame_id>
+		</plugin>
+	</gazebo>
+	<gazebo>
+		<plugin filename="gz-sim-joint-state-publisher-system" name="gz::sim::systems::JointStatePublisher">
+			<topic>joint_states</topic>
+			<joint_name>front_left_wheel_joint</joint_name>
+			<joint_name>rear_left_wheel_joint</joint_name>
+			<joint_name>front_right_wheel_joint</joint_name>
+			<joint_name>rear_right_wheel_joint</joint_name>
+		</plugin>
+	</gazebo>
+	<xacro:macro name="wheel_gazebo" params="name">
+		<gazebo reference="${name}">
+			<mu1>1.0</mu1>
+			<mu2>1.0</mu2>
+			<kp>1e6</kp>
+			<kd>1.0</kd>
+			<minDepth>0.001</minDepth>
+		</gazebo>
+	</xacro:macro>
+	<xacro:wheel_gazebo name="front_left_wheel"/>
+	<xacro:wheel_gazebo name="rear_left_wheel"/>
+	<xacro:wheel_gazebo name="front_right_wheel"/>
+	<xacro:wheel_gazebo name="rear_right_wheel"/>
+</robot>
